File: placa.kicad_pcb (KiCad board)
At the start: 2 copper layers, 40 x 40 mm, 74 parts, among them J1 SW, J10 CONN_01X04_Straight, J11 CONN_01X04_Straight, J12 CONN_01X04_Straight, J13 CONN_01X04_Straight, J2 μUSB, J3 BATT, J6 CONN_01X12_Straight, J7 CONN_02X12_Straight, J8 CONN_01X04_Straight, J9 CONN_01X04_Straight, Q1 BSS84, Q2 BSS138P, Q3 BSS138P, U1 AP2112K-3.3TRG1, U2 MCP73831, U3 MIC2253-06YML-TR, U4 ADS1000, U5 LMC7101AIM5, U6 DRV8837, U7 DRV8837, U8 PCA9670

Commit message: Board
Parts:
- L1: value HPI0630-2R2 -> HPI0530-2R2; footprint alvaroferran:HPI0630-2R2 -> alvaroferran:HPI0530-2R2
- moved L1 1.89 mm to (159.8, 85.4)
- moved D3 1.60 mm to (164.6, 84.3)
- moved C12 0.51 mm to (164.1, 83.8)
- moved C13 0.51 mm to (164.1, 80.8)
- moved C8 0.51 mm to (164.1, 85.3)
- moved C9 0.51 mm to (164.1, 86.9)
- moved R16 0.51 mm to (164.1, 88.4)
- moved R17 0.51 mm to (164.1, 82.3)
- moved R4 0.51 mm to (164.1, 79.2)
Connections:
- J2 pad 2: (no net) -> Net-(J2-Pad2)
- J2 pad 3: (no net) -> Net-(J2-Pad3)
- J2 pad 4: (no net) -> Net-(J2-Pad4)
- J6 pad 1: (no net) -> Net-(J6-Pad1)
- J6 pad 10: (no net) -> Net-(J6-Pad10)
- J6 pad 11: (no net) -> Net-(J6-Pad11)
- J6 pad 2: (no net) -> Net-(J6-Pad2)
- J6 pad 3: (no net) -> Net-(J6-Pad3)
- J6 pad 6: (no net) -> Net-(J6-Pad6)
- J6 pad 7: (no net) -> Net-(J6-Pad7)
- J6 pad 8: (no net) -> Net-(J6-Pad8)
- J6 pad 9: (no net) -> Net-(J6-Pad9)
- J7 pad 1: (no net) -> Net-(J7-Pad1)
- J7 pad 10: (no net) -> Net-(J7-Pad10)
- J7 pad 11: (no net) -> Net-(J7-Pad11)
- J7 pad 12: (no net) -> Net-(J7-Pad12)
- J7 pad 13: (no net) -> Net-(J7-Pad13)
- J7 pad 15: (no net) -> Net-(J7-Pad15)
- J7 pad 16: (no net) -> Net-(J7-Pad16)
- J7 pad 17: (no net) -> Net-(J7-Pad17)
- J7 pad 18: (no net) -> Net-(J7-Pad18)
- J7 pad 19: (no net) -> Net-(J7-Pad19)
- J7 pad 21: (no net) -> Net-(J7-Pad21)
- J7 pad 22: (no net) -> Net-(J7-Pad22)
- J7 pad 23: (no net) -> Net-(J7-Pad23)
- J7 pad 24: (no net) -> Net-(J7-Pad24)
- J7 pad 7: (no net) -> Net-(J7-Pad7)
- J7 pad 8: (no net) -> Net-(J7-Pad8)
- U1 pad 4: (no net) -> Net-(U1-Pad4)
- U3 pad 1: (no net) -> Net-(U3-Pad1)
Routing:
- net GND: track 0.00 -> 95.9 mm
- net 5V: track 0.00 -> 25.0 mm, vias 0 -> 1
- net VBAT: track 0.00 -> 23.7 mm, vias 0 -> 1
- net Net-(D4-Pad1): track 0.00 -> 15.3 mm, vias 0 -> 1
- net Net-(D3-Pad2): track 0.00 -> 11.6 mm, vias 0 -> 1
- net GNDA: track 0.00 -> 10.2 mm, vias 0 -> 2
- net Net-(C7-Pad2): track 0.00 -> 10.1 mm
- net Net-(R10-Pad2): track 0.00 -> 7.21 mm
- net GNDPWR: track 0.00 -> 6.14 mm
- net Net-(C12-Pad2): track 0.00 -> 3.64 mm, vias 0 -> 2
- net Net-(C13-Pad1): track 0.00 -> 3.13 mm
- net (no net): track 1.74 -> 0.00 mm
Other:
- rule trace_min: 0.2 -> 0.1524

Commit message: Board
Parts:
- removed JP2: Jumper_NO, Connectors:GS2
- moved C8 5.71 mm to (159.3, 88.4), turned to 0 degrees
- moved C9 1.65 mm to (164.1, 85.2)
- moved R16 1.40 mm to (164.1, 87.0)
- moved C1 1.14 mm to (169.2, 83.6), turned to 270 degrees
- moved C2 0.76 mm to (168.9, 77.5)
- moved C4 0.76 mm to (171.7, 77.5)
- moved C3 0.57 mm to (171.2, 83.6), turned to 270 degrees
- moved U1 0.51 mm to (170.2, 80.3)
Routing:
- net 5V: track 25.0 -> 77.2 mm, vias 1 -> 2
- net /SCL: track 0.00 -> 20.9 mm
- net Net-(C5-Pad1): track 0.00 -> 19.7 mm, vias 0 -> 2
- net /GPIO3: track 0.00 -> 16.7 mm
- net /GPIO2: track 0.00 -> 15.3 mm
- net /SDAH: track 0.00 -> 14.0 mm, vias 0 -> 1
- net /SCLH: track 0.00 -> 12.3 mm, vias 0 -> 1
- net /GPIO1: track 0.00 -> 11.5 mm
- net VBAT: track 23.7 -> 33.6 mm, vias 1 -> 2
- net Net-(JP2-Pad1): track 0.00 -> 7.15 mm, vias 0 -> 1
- net /GPIO0: track 0.00 -> 6.65 mm
- net Net-(JP3-Pad1): track 0.00 -> 4.58 mm, vias 0 -> 1
- net Net-(C6-Pad1): track 0.00 -> 4.35 mm
- net Net-(JP1-Pad1): track 0.00 -> 3.89 mm, vias 0 -> 1
- net 3.3V: track 0.00 -> 3.33 mm
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
Commit message: Board
Parts:
- added JP2: Jumper_NO, Connectors:GS2, B.Cu at (174.5, 89.9)
- moved R1 4.83 mm to (179.6, 76.5), turned to 180 degrees
- moved D1 3.25 mm to (176.8, 76.5), turned to 180 degrees
- moved R8 1.14 mm to (152.9, 83.6), turned to 180 degrees
- moved R15 1.08 mm to (150.9, 82.3), turned to 180 degrees
- moved R14 0.80 mm to (152.9, 82.3), turned to 0 degrees
- moved R9 0.72 mm to (150.9, 83.6), turned to 0 degrees
- moved U4 0.57 mm to (151.9, 79.8)
- moved C18 0.51 mm to (171.4, 85.6)
- moved U6 0.25 mm to (178.6, 92.7)
- moved U7 0.25 mm to (178.6, 86.9)
- moved C14 0.25 mm to (177.5, 89.2)
- moved C15 0.25 mm to (179.6, 89.2)
- moved C16 0.25 mm to (177.5, 95.0)
- moved C17 0.25 mm to (179.6, 95.0)
Connections:
- J2 pad 2: Net-(J2-Pad2) -> (no net)
- J2 pad 3: Net-(J2-Pad3) -> (no net)
- J2 pad 4: Net-(J2-Pad4) -> (no net)
- J6 pad 1: Net-(J6-Pad1) -> (no net)
- J6 pad 10: Net-(J6-Pad10) -> (no net)
- J6 pad 11: Net-(J6-Pad11) -> (no net)
- J6 pad 2: Net-(J6-Pad2) -> (no net)
- J6 pad 3: Net-(J6-Pad3) -> (no net)
- J6 pad 6: Net-(J6-Pad6) -> (no net)
- J6 pad 7: Net-(J6-Pad7) -> (no net)
- J6 pad 8: Net-(J6-Pad8) -> (no net)
- J6 pad 9: Net-(J6-Pad9) -> (no net)
- J7 pad 1: Net-(J7-Pad1) -> (no net)
- J7 pad 10: Net-(J7-Pad10) -> (no net)
- J7 pad 11: Net-(J7-Pad11) -> (no net)
- J7 pad 12: Net-(J7-Pad12) -> (no net)
- J7 pad 13: Net-(J7-Pad13) -> (no net)
- J7 pad 15: Net-(J7-Pad15) -> (no net)
- J7 pad 16: Net-(J7-Pad16) -> (no net)
- J7 pad 17: Net-(J7-Pad17) -> (no net)
- J7 pad 18: Net-(J7-Pad18) -> (no net)
- J7 pad 19: Net-(J7-Pad19) -> (no net)
- J7 pad 21: Net-(J7-Pad21) -> (no net)
- J7 pad 22: Net-(J7-Pad22) -> (no net)
- J7 pad 23: Net-(J7-Pad23) -> (no net)
- J7 pad 24: Net-(J7-Pad24) -> (no net)
- J7 pad 7: Net-(J7-Pad7) -> (no net)
- J7 pad 8: Net-(J7-Pad8) -> (no net)
- U1 pad 4: Net-(U1-Pad4) -> (no net)
- U3 pad 1: Net-(U3-Pad1) -> (no net)
Routing:
- net 5V: track 77.2 -> 155.6 mm, vias 2 -> 7
- net /SDA: track 0.00 -> 63.6 mm, vias 0 -> 2
- net 3.3V: track 3.33 -> 60.3 mm, vias 0 -> 5
- net /SCL: track 20.9 -> 67.4 mm
- net Net-(C6-Pad1): track 4.35 -> 44.2 mm, vias 0 -> 1
- net GND: track 98.5 -> 134.9 mm, vias 11 -> 53
- net VBAT: track 33.6 -> 59.6 mm, vias 2 -> 3
- net /MOTEN: track 0.00 -> 18.2 mm, vias 0 -> 2
- net Net-(J4-Pad1): track 0.00 -> 6.28 mm, vias 0 -> 1
- net Net-(J5-Pad1): track 0.00 -> 6.18 mm, vias 0 -> 1
- net Net-(J4-Pad2): track 0.00 -> 6.18 mm, vias 0 -> 1
- net Net-(J5-Pad2): track 0.00 -> 6.07 mm, vias 0 -> 1
- net /MOT1A: track 0.00 -> 5.03 mm
- net /MOT2B: track 0.00 -> 4.43 mm
- net Net-(R12-Pad1): track 0.00 -> 3.24 mm
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
Commit message: Board
Routing:
- net 3.3V: track 60.3 -> 112.7 mm, vias 5 -> 7
- net Net-(Q1-Pad1): track 0.00 -> 4.76 mm, vias 0 -> 2
- net 5V: track 155.6 -> 159.6 mm
- net GND: track 134.9 -> 137.4 mm, vias 53 -> 92
- net Net-(D3-Pad2): track 12.2 -> 13.2 mm
