File: placa.kicad_pcb (KiCad board)
At the start: 2 copper layers, 40 x 40 mm, 74 parts, among them J1 SW, J10 CONN_01X04_Straight, J11 CONN_01X04_Straight, J12 CONN_01X04_Straight, J13 CONN_01X04_Straight, J2 μUSB, J3 BATT, J6 CONN_01X12_Straight, J7 CONN_02X12_Straight, J8 CONN_01X04_Straight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

Commit message: Board
Routing:
- net Net-(D4-Pad1): track 15.3 -> 8.68 mm, vias 1 -> 0
- net Net-(C5-Pad1): track 19.7 -> 19.2 mm
- net GND: vias 92 -> 109
