File: KiCad/neoBoard.kicad_pcb (KiCad board)
At the start: 2 copper layers, 40 x 40 mm, 74 parts, among them J1 SW, J10 CONN_01X04_Straight, J11 CONN_01X04_Straight, J12 CONN_01X04_Straight, J13 CONN_01X04_Straight, J2 μUSB, J3 BATT, J6 CONN_01X12_Straight, J7 CONN_02X12_Straight, J8 CONN_01X04_Straight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

Commit message: Board
Routing:
- net 3.3V: track 112.3 -> 113.0 mm
- net GND: vias 109 -> 116
Other:
- net class Default: clearance 0.2 -> 0
- rule trace_clearance: 0.2 -> 0
- board text added: "NEO BOARD"
- board text removed: "BOARD NAME"
